File: EP6/Electrical_Group/Dash_Screen/Dash_Screen.kicad_sch (KiCad schematic)
At the start: 29 parts, among them J10 BUT5, J13 BUT6, J14 BUT7, J15 RTD_LED, J3 VCU, J4 12864, J5 toLCD, J6 BUT1, J7 BUT2, J8 BUT3, J9 BUT4, Q1 2N7002, Q2 AO3401A

Commit message: update Dash_Screen to V1.0
Other:
- title: EP6 Dash screen -> Dash_screen
Changed lines of the file:
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@@
 	(paper "A4")
 	(title_block
-		(title "EP6 Dash screen")
+		(title "Dash_screen")
 		(date "2025-03-07")
 		(rev "1.0")
