File: EP6/Powertrain_Group/ACC_BMSslave/tprobe_mux.kicad_sch (KiCad schematic)
At the start: 2 parts, among them U3 ADG758CPZ

Commit message: ACC_BMSslave pcb priliminary layout
Parts:
- C24: footprint Capacitor_SMD:C_0201_0603Metric -> Capacitor_SMD:C_0603_1608Metric
Connections:
- net T1: now also U3.13 (S5); no longer U3.3 (S1)
- net T2: now also U3.12 (S6); no longer U3.4 (S2)
- net T3: now also U3.11 (S7); no longer U3.5 (S3)
- net T4: now also U3.10 (S8); no longer U3.6 (S4)
- net T5: now also U3.6 (S4); no longer U3.13 (S5)
- net T6: now also U3.5 (S3); no longer U3.12 (S6)
- net T7: now also U3.4 (S2); no longer U3.11 (S7)
- net T8: now also U3.3 (S1); no longer U3.10 (S8)
Changed lines of the file:
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@@
 		)
 	)
-	(hierarchical_label "T7"
+	(hierarchical_label "T3"
 		(shape input)
 		(at 93.98 96.52 180)
@@
 		)
 	)
-	(hierarchical_label "T1"
+	(hierarchical_label "T8"
 		(shape input)
 		(at 93.98 81.28 180)
@@
 		)
 	)
-	(hierarchical_label "T3"
+	(hierarchical_label "T6"
 		(shape input)
 		(at 93.98 86.36 180)
@@
 		)
 	)
-	(hierarchical_label "T2"
+	(hierarchical_label "T7"
 		(shape input)
 		(at 93.98 83.82 180)
@@
 		)
 	)
-	(hierarchical_label "T4"
+	(hierarchical_label "T5"
 		(shape input)
 		(at 93.98 88.9 180)
@@
 		)
 	)
-	(hierarchical_label "T8"
+	(hierarchical_label "T4"
 		(shape input)
 		(at 93.98 99.06 180)
@@
 		)
 	)
-	(hierarchical_label "T6"
+	(hierarchical_label "T2"
 		(shape input)
 		(at 93.98 93.98 180)
@@
 		)
 	)
-	(hierarchical_label "T5"
+	(hierarchical_label "T1"
 		(shape input)
 		(at 93.98 91.44 180)
@@
 			)
 		)
-		(property "Footprint" "Capacitor_SMD:C_0201_0603Metric"
+		(property "Footprint" "Capacitor_SMD:C_0603_1608Metric"
 			(at 119.38 63.5 0)
 			(effects

Commit message: ACC_BMSslave snapshot
Parts:
- removed U3: ADG758CPZ, Package_CSP:LFCSP-20-1EP_4x4mm_P0.5mm_EP2.1x2.1mm, symbol Analog_Switch:ADG758CPZ
- added U4: CD4051B, Package_SO:TSSOP-16_4.4x5mm_P0.65mm, symbol Analog_Switch:CD4051B
- renumbered C24 to C23
Connections:
- net A0: now also U4.11 (A)
- net A1: now also U4.10 (B)
- net A2: now also U4.9 (C)
- net Earth: now also U4.6 (INH), U4.7 (VEE), U4.8 (VSS)
- net OUT: now also U4.3 (X)
- net T1: now also U4.1 (X4)
- net T2: now also U4.5 (X5)
- net T3: now also U4.2 (X6)
- net T4: now also U4.4 (X7)
- net T5: now also U4.12 (X3)
- net T6: now also U4.15 (X2)
- net T7: now also U4.14 (X1)
- net T8: now also U4.13 (X0)
- net VREG: now also U4.16 (VDD)
Other:
- moved on the sheet: C23

Commit message: ACC_BMSslave snapshot
Parts:
- renumbered U4 to U3
Connections:
- net T1: now also U3.13 (X0); no longer U3.1 (X4)
- net T2: now also U3.14 (X1); no longer U3.5 (X5)
- net T3: now also U3.15 (X2); no longer U3.2 (X6)
- net T4: now also U3.12 (X3); no longer U3.4 (X7)
- net T5: now also U3.1 (X4); no longer U3.12 (X3)
- net T6: now also U3.5 (X5); no longer U3.15 (X2)
- net T7: now also U3.2 (X6); no longer U3.14 (X1)
- net T8: now also U3.4 (X7); no longer U3.13 (X0)
Changed lines of the file:
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@@
 	(hierarchical_label "T3"
 		(shape input)
+		(at 161.29 81.28 0)
+		(fields_autoplaced yes)
+		(effects
+			(font
+				(size 1.27 1.27)
+			)
+			(justify left)
+		)
+	)
+	(hierarchical_label "T8"
+		(shape input)
+		(at 161.29 93.98 0)
+		(fields_autoplaced yes)
+		(effects
+			(font
+				(size 1.27 1.27)
+			)
+			(justify left)
+		)
+	)
+	(hierarchical_label "T6"
+		(shape input)
+		(at 161.29 88.9 0)
+		(fields_autoplaced yes)
+		(effects
+			(font
+				(size 1.27 1.27)
+			)
+			(justify left)
+		)
+	)
+	(hierarchical_label "A2"
+		(shape input)
+		(at 133.35 73.66 180)
+		(fields_autoplaced yes)
+		(effects
+			(font
+				(size 1.27 1.27)
+			)
+			(justify right)
+		)
+	)
+	(hierarchical_label "T7"
+		(shape input)
 		(at 161.29 91.44 0)
 		(fields_autoplaced yes)
@@
 		)
 	)
-	(hierarchical_label "T8"
-		(shape input)
-		(at 161.29 76.2 0)
-		(fields_autoplaced yes)
-		(effects
-			(font
-				(size 1.27 1.27)
-			)
-			(justify left)
-		)
-	)
-	(hierarchical_label "T6"
-		(shape input)
-		(at 161.29 81.28 0)
-		(fields_autoplaced yes)
-		(effects
-			(font
-				(size 1.27 1.27)
-			)
-			(justify left)
-		)
-	)
-	(hierarchical_label "A2"
-		(shape input)
-		(at 133.35 73.66 180)
-		(fields_autoplaced yes)
-		(effects
-			(font
-				(size 1.27 1.27)
-			)
-			(justify right)
-		)
-	)
-	(hierarchical_label "T7"
+	(hierarchical_label "T5"
+		(shape input)
+		(at 161.29 86.36 0)
+		(fields_autoplaced yes)
+		(effects
+			(font
+				(size 1.27 1.27)
+			)
+			(justify left)
+		)
+	)
+	(hierarchical_label "T4"
+		(shape input)
+		(at 161.29 83.82 0)
+		(fields_autoplaced yes)
+		(effects
+			(font
+				(size 1.27 1.27)
+			)
+			(justify left)
+		)
+	)
+	(hierarchical_label "T2"
 		(shape input)
 		(at 161.29 78.74 0)
-		(fields_autoplaced yes)
-		(effects
-			(font
-				(size 1.27 1.27)
-			)
-			(justify left)
-		)
-	)
-	(hierarchical_label "T5"
-		(shape input)
-		(at 161.29 83.82 0)
-		(fields_autoplaced yes)
-		(effects
-			(font
-				(size 1.27 1.27)
-			)
-			(justify left)
-		)
-	)
-	(hierarchical_label "T4"
-		(shape input)
-		(at 161.29 93.98 0)
-		(fields_autoplaced yes)
-		(effects
-			(font
-				(size 1.27 1.27)
-			)
-			(justify left)
-		)
-	)
-	(hierarchical_label "T2"
-		(shape input)
-		(at 161.29 88.9 0)
 		(fields_autoplaced yes)
 		(effects
@@
 	(hierarchical_label "T1"
 		(shape input)
-		(at 161.29 86.36 0)
+		(at 161.29 76.2 0)
 		(fields_autoplaced yes)
 		(effects
@@
 		(instances
 			(project "ACC_BMSslave"
-				(path "/0942010f-46b1-4fe9-9f5e-a3ebd22b3e41/211e644c-7f46-49c6-a3f8-aa27bfb858de"
-					(reference "C59")
+				(path "/0942010f-46b1-4fe9-9f5e-a3ebd22b3e41/10788a82-4d92-4105-8ade-edb24ffdc07f"
+					(reference "C26")
 					(unit 1)
 				)
@@
 					(unit 1)
 				)
-				(path "/0942010f-46b1-4fe9-9f5e-a3ebd22b3e41/9183c6cf-6611-4bb2-b245-fcd870ea1106"
-					(reference "C60")
-					(unit 1)
-				)
 				(path "/0942010f-46b1-4fe9-9f5e-a3ebd22b3e41/adcc2476-b4f7-4052-a515-98c15e743abf"
 					(reference "C24")
-					(unit 1)
-				)
-				(path "/0942010f-46b1-4fe9-9f5e-a3ebd22b3e41/f8a4b11f-3e41-4868-8c26-04590eafeccb"
-					(reference "C61")
 					(unit 1)
 				)
@@
 		(instances
 			(project "ACC_BMSslave"
-				(path "/0942010f-46b1-4fe9-9f5e-a3ebd22b3e41/211e644c-7f46-49c6-a3f8-aa27bfb858de"
-					(reference "#PWR098")
+				(path "/0942010f-46b1-4fe9-9f5e-a3ebd22b3e41/10788a82-4d92-4105-8ade-edb24ffdc07f"
+					(reference "#PWR041")
 					(unit 1)
 				)
@@
 					(unit 1)
 				)
-				(path "/0942010f-46b1-4fe9-9f5e-a3ebd22b3e41/9183c6cf-6611-4bb2-b245-fcd870ea1106"
-					(reference "#PWR0102")
-					(unit 1)
-				)
 				(path "/0942010f-46b1-4fe9-9f5e-a3ebd22b3e41/adcc2476-b4f7-4052-a515-98c15e743abf"
 					(reference "#PWR066")
-					(unit 1)
-				)
-				(path "/0942010f-46b1-4fe9-9f5e-a3ebd22b3e41/f8a4b11f-3e41-4868-8c26-04590eafeccb"
-					(reference "#PWR0106")
 					(unit 1)
 				)
@@
 		(dnp no)
 		(fields_autoplaced yes)
-		(property "Reference" "U4"
+		(property "Reference" "U3"
 			(at 152.0541 60.96 0)
 			(effects
@@
 		(instances
 			(project "ACC_BMSslave"
-				(path "/0942010f-46b1-4fe9-9f5e-a3ebd22b3e41/211e644c-7f46-49c6-a3f8-aa27bfb858de"
+				(path "/0942010f-46b1-4fe9-9f5e-a3ebd22b3e41/10788a82-4d92-4105-8ade-edb24ffdc07f"
 					(reference "U6")
 					(unit 1)
@@
 					(unit 1)
 				)
-				(path "/0942010f-46b1-4fe9-9f5e-a3ebd22b3e41/9183c6cf-6611-4bb2-b245-fcd870ea1106"
-					(reference "U7")
-					(unit 1)
-				)
 				(path "/0942010f-46b1-4fe9-9f5e-a3ebd22b3e41/adcc2476-b4f7-4052-a515-98c15e743abf"
 					(reference "U4")
-					(unit 1)
-				)
-				(path "/0942010f-46b1-4fe9-9f5e-a3ebd22b3e41/f8a4b11f-3e41-4868-8c26-04590eafeccb"
-					(reference "U8")
 					(unit 1)
 				)
@@
 		(instances
 			(project "ACC_BMSslave"
-				(path "/0942010f-46b1-4fe9-9f5e-a3ebd22b3e41/211e644c-7f46-49c6-a3f8-aa27bfb858de"
-					(reference "#PWR0100")
+				(path "/0942010f-46b1-4fe9-9f5e-a3ebd22b3e41/10788a82-4d92-4105-8ade-edb24ffdc07f"
+					(reference "#PWR095")
 					(unit 1)
 				)
@@
 					(unit 1)
 				)
-				(path "/0942010f-46b1-4fe9-9f5e-a3ebd22b3e41/9183c6cf-6611-4bb2-b245-fcd870ea1106"
-					(reference "#PWR0104")
-					(unit 1)
-				)
 				(path "/0942010f-46b1-4fe9-9f5e-a3ebd22b3e41/adcc2476-b4f7-4052-a515-98c15e743abf"
 					(reference "#PWR068")
-					(unit 1)
-				)
-				(path "/0942010f-46b1-4fe9-9f5e-a3ebd22b3e41/f8a4b11f-3e41-4868-8c26-04590eafeccb"
-					(reference "#PWR0108")
 					(unit 1)
 				)
@@
 		(instances
 			(project "ACC_BMSslave"
-				(path "/0942010f-46b1-4fe9-9f5e-a3ebd22b3e41/211e644c-7f46-49c6-a3f8-aa27bfb858de"
-					(reference "#PWR0101")
+				(path "/0942010f-46b1-4fe9-9f5e-a3ebd22b3e41/10788a82-4d92-4105-8ade-edb24ffdc07f"
+					(reference "#PWR096")
 					(unit 1)
 				)
@@
 					(unit 1)
 				)
-				(path "/0942010f-46b1-4fe9-9f5e-a3ebd22b3e41/9183c6cf-6611-4bb2-b245-fcd870ea1106"
-					(reference "#PWR0105")
-					(unit 1)
-				)
 				(path "/0942010f-46b1-4fe9-9f5e-a3ebd22b3e41/adcc2476-b4f7-4052-a515-98c15e743abf"
 					(reference "#PWR069")
-					(unit 1)
-				)
-				(path "/0942010f-46b1-4fe9-9f5e-a3ebd22b3e41/f8a4b11f-3e41-4868-8c26-04590eafeccb"
-					(reference "#PWR0109")
 					(unit 1)
 				)
@@
 		(instances
 			(project "ACC_BMSslave"
-				(path "/0942010f-46b1-4fe9-9f5e-a3ebd22b3e41/211e644c-7f46-49c6-a3f8-aa27bfb858de"
-					(reference "#PWR099")
+				(path "/0942010f-46b1-4fe9-9f5e-a3ebd22b3e41/10788a82-4d92-4105-8ade-edb24ffdc07f"
+					(reference "#PWR074")
 					(unit 1)
 				)
@@
 					(unit 1)
 				)
-				(path "/0942010f-46b1-4fe9-9f5e-a3ebd22b3e41/9183c6cf-6611-4bb2-b245-fcd870ea1106"
-					(reference "#PWR0103")
-					(unit 1)
-				)
 				(path "/0942010f-46b1-4fe9-9f5e-a3ebd22b3e41/adcc2476-b4f7-4052-a515-98c15e743abf"
 					(reference "#PWR067")
 					(unit 1)
 				)
-				(path "/0942010f-46b1-4fe9-9f5e-a3ebd22b3e41/f8a4b11f-3e41-4868-8c26-04590eafeccb"
-					(reference "#PWR0107")
-					(unit 1)
-				)

Commit message: [BMSslave] snapshot
Parts:
- added C1: 100n, Capacitor_SMD:C_0603_1608Metric, symbol Device:C_Small
- added R1, R2, R3, R4, R5, R6, R7, R8: 4k3, Resistor_SMD:R_0402_1005Metric, symbol Device:R_Small
- renumbered C23 to C26, U3 to U6
Connections:
- net Earth: now also C1.2
- net T1: now also R1.1
- net T2: now also R2.1
- net T3: now also R3.1
- net T4: now also R4.1
- net T5: now also R5.1
- net T6: now also R6.1
- net T7: now also R7.1
- net T8: now also R8.1
- new net VREF: C1.1, R1.2, R2.2, R3.2, R4.2, R5.2, R6.2, R7.2, R8.2

Commit message: [BMSslave] snapshot
Parts:
- C25: renamed from C26; value 10n -> 100n; footprint Capacitor_SMD:C_0603_1608Metric -> Capacitor_SMD:C_0402_1005Metric
- C26: renamed from C1; footprint Capacitor_SMD:C_0603_1608Metric -> Capacitor_SMD:C_0402_1005Metric
- renumbered R1 to R47, R2 to R48, R3 to R49, R4 to R50, R5 to R51, R6 to R52, R7 to R53, R8 to R54, U6 to U5

Commit message: [BMSslave] snapshot
Parts:
- renumbered C25 to C19, C26 to C20, R47 to R20, R48 to R21, R49 to R22, R50 to R23, R51 to R24, R52 to R25, R53 to R26, R54 to R27, U5 to U2

Commit message: [BMSslave] initial layout
Parts:
- R20, R21, R22, R23, R24, R25, R26, R27: value 4k3 -> 10k
Changed lines of the file:
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@@
 			)
 		)
-		(property "Value" "4k3"
+		(property "Value" "10k"
 			(at 205.74 109.22 90)
 			(effects
@@
 			)
 		)
-		(property "Value" "4k3"
+		(property "Value" "10k"
 			(at 205.74 93.98 90)
 			(effects
@@
 			)
 		)
-		(property "Value" "4k3"
+		(property "Value" "10k"
 			(at 205.74 73.66 90)
 			(effects
@@
 			)
 		)
-		(property "Value" "4k3"
+		(property "Value" "10k"
 			(at 205.74 78.74 90)
 			(effects
@@
 			)
 		)
-		(property "Value" "4k3"
+		(property "Value" "10k"
 			(at 205.74 88.9 90)
 			(effects
@@
 			)
 		)
-		(property "Value" "4k3"
+		(property "Value" "10k"
 			(at 205.74 104.14 90)
 			(effects
@@
 			)
 		)
-		(property "Value" "4k3"
+		(property "Value" "10k"
 			(at 205.74 83.82 90)
 			(effects
@@
 			)
 		)
-		(property "Value" "4k3"
+		(property "Value" "10k"
 			(at 205.74 99.06 90)
 			(effects
