File: EP6/Electrical_Group/RPI_diyhat1/RPI_diyhat1.kicad_pcb (KiCad board)
At the start: 2 copper layers, 65 x 56 mm, 81 parts, among them IC1 LSM303AGRTR, IC3 LSF0204DPWR, J1 Raspberry_Pi_2_3, J2 CAN2, J3 LVBattery, J4 LVBattery, J5 CAN2, U1 TPS5430DDAR, U2 MCP2515-xSO, U3 MCP7940N-xSN, U4 TCAN1042VDRQ1, U5 LSM6DSOX, U6 AMS1117-3.3, Y1 32.768kHz Q13FC13500004, Y2 8MHz X49SM8MSD2SC

Commit message: update RPI_diyhat1 to V1.2
Parts:
- removed C12: 30p, Capacitor_SMD:C_0402_1005Metric
- removed C17, C18: 100n, Capacitor_SMD:C_0402_1005Metric
- removed D2: GREEN CANopen_RUN, LED_SMD:LED_0603_1608Metric
- removed D4: RED CANopen_ERR, LED_SMD:LED_0603_1608Metric
- removed IC3: LSF0204DPWR, SamacSys_Parts_EP6:SOP65P640X120-14N
- removed TP1: CAN RUN, TestPoint:TestPoint_Pad_D1.0mm
- removed TP2: CAN ERR, TestPoint:TestPoint_Pad_D1.0mm
- added C10: 100n, Capacitor_SMD:C_0603_1608Metric, F.Cu at (141.6, 124.5)
- added C34: 100n, Capacitor_SMD:C_0603_1608Metric, F.Cu at (151.0, 107.9)
- added C35: 100n, Capacitor_SMD:C_0603_1608Metric, F.Cu at (149.0, 117.7)
- added C48: 30p, Capacitor_SMD:C_0603_1608Metric, F.Cu at (147.3, 86.8)
- added C49: 30p, Capacitor_SMD:C_0603_1608Metric, F.Cu at (142.2, 86.8)
- added C50: 30p, Capacitor_SMD:C_0603_1608Metric, F.Cu at (147.3, 106.7)
- added C51: 30p, Capacitor_SMD:C_0603_1608Metric, F.Cu at (142.2, 106.7)
- added D8: NUP2105L, Package_TO_SOT_SMD:SOT-23, F.Cu at (151.5, 118.1)
- added J6: CAN2, Connector_JST:JST_XH_B2B-XH-A_1x02_P2.50mm_Vertical, F.Cu at (157.1, 118.7)
- added J7: CAN2, Connector_JST:JST_XH_B2B-XH-A_1x02_P2.50mm_Vertical, F.Cu at (157.1, 110.2)
- added R15: 0R, Resistor_SMD:R_0603_1608Metric, F.Cu at (131.0, 102.9)
- added R16: 0R, Resistor_SMD:R_0603_1608Metric, F.Cu at (129.0, 102.9)
- added R17: 10k, Resistor_SMD:R_0603_1608Metric, F.Cu at (145.0, 120.0)
- added R18: 10k, Capacitor_SMD:C_0603_1608Metric, F.Cu at (151.0, 105.5)
- added R19: 0R, Resistor_SMD:R_0402_1005Metric, F.Cu at (137.0, 119.5)
- added R20: 0R, Resistor_SMD:R_0603_1608Metric, F.Cu at (130.5, 108.0)
- added R25: 0R, Resistor_SMD:R_0603_1608Metric, F.Cu at (136.7, 91.7)
- added R26: 0R, Resistor_SMD:R_0603_1608Metric, F.Cu at (134.7, 91.7)
- added R27: 0R, Resistor_SMD:R_0603_1608Metric, F.Cu at (125.4, 91.7)
- added R28: 0R, Resistor_SMD:R_0603_1608Metric, F.Cu at (123.4, 91.7)
- added R29: 0R, Resistor_SMD:R_0603_1608Metric, F.Cu at (132.0, 97.5)
- added R30: 0R, Resistor_SMD:R_0603_1608Metric, F.Cu at (128.0, 97.5)
- added R31: 0R, Resistor_SMD:R_0603_1608Metric, F.Cu at (125.4, 97.5)
- added R32: 0R, Resistor_SMD:R_0603_1608Metric, F.Cu at (123.4, 97.5)
- added R33: 0R, Resistor_SMD:R_0603_1608Metric, F.Cu at (131.0, 91.7)
- added R34: 0R, Resistor_SMD:R_0603_1608Metric, F.Cu at (129.0, 91.7)
- added R35: 0R, Resistor_SMD:R_0603_1608Metric, F.Cu at (130.0, 97.5)
- added U12: MCP2515-xST, Package_SO:TSSOP-20_4.4x6.5mm_P0.65mm, F.Cu at (144.7, 94.0)
- added U13: MCP2515-xST, Package_SO:TSSOP-20_4.4x6.5mm_P0.65mm, F.Cu at (144.7, 113.9)
- added U8: TCAN1042VDRQ1, Package_SO:SOIC-8_3.9x4.9mm_P1.27mm, F.Cu at (151.0, 112.5)
- added Y3: 12MHz 830105420809, Crystal:Crystal_SMD_3225-4Pin_3.2x2.5mm, F.Cu at (144.7, 107.3)
- BT1: moved to B.Cu
- C1: value 10u 35V -> 100n; footprint Capacitor_SMD:C_1206_3216Metric -> Capacitor_SMD:C_0402_1005Metric
- C11, C15, C16, C9: value 0u1 -> 100n
- C13, C14: value 0u1 -> 100n; footprint Capacitor_SMD:C_0402_1005Metric -> Capacitor_SMD:C_0603_1608Metric
- C2, C3: footprint Capacitor_SMD:C_0402_1005Metric -> Capacitor_SMD:C_0603_1608Metric
- C6: value 220u 35V -> 100u 25V; footprint Capacitor_THT:CP_Radial_D8.0mm_P3.80mm -> Capacitor_THT:CP_Radial_D6.3mm_P2.50mm
- C7: value 220u 35V -> 100u 35V; footprint Capacitor_THT:CP_Radial_D8.0mm_P3.80mm -> Capacitor_THT:CP_Radial_D6.3mm_P2.50mm
- C8: value 30p -> 100n
- D7: value RED 3V3 -> WHITE LED
- F3: value 3A -> 3V3 FUSE
- R1: value 47k 1% -> 18k
- R10, R9: value 3k3 -> 1k
- R12, R6: footprint Resistor_SMD:R_0402_1005Metric -> Resistor_SMD:R_0603_1608Metric
- R13: value 1k -> 10k; footprint Resistor_SMD:R_0402_1005Metric -> Resistor_SMD:R_0603_1608Metric
- R14: value 510R -> 10k; footprint Resistor_SMD:R_0402_1005Metric -> Resistor_SMD:R_0603_1608Metric
- R2: value 15k 1% -> 5k6
- R3, R5: value 1k -> 0R; footprint Resistor_SMD:R_0402_1005Metric -> Resistor_SMD:R_0603_1608Metric
- R4: footprint Resistor_SMD:R_0402_1005Metric -> Capacitor_SMD:C_0603_1608Metric
- R8: value 20R -> 0R; footprint Resistor_SMD:R_0402_1005Metric -> Resistor_SMD:R_0603_1608Metric
- U2: value MCP2515-xSO -> LSM6DSOX; footprint Package_SO:SOIC-18W_7.5x11.6mm_P1.27mm -> Package_LGA:LGA-14_3x2.5mm_P0.5mm_LayoutBorder3x4y
- Y2: value 8MHz X49SM8MSD2SC -> 12MHz 830105420809; footprint Crystal:Crystal_SMD_5032-2Pin_5.0x3.2mm -> Crystal:Crystal_SMD_3225-4Pin_3.2x2.5mm
- moved C8 36.5 mm to (135.2, 116.6), turned to 0 degrees
- moved C1 34.7 mm to (133.3, 116.6)
- moved C2 34.1 mm to (147.5, 119.5), turned to 90 degrees
- moved R9 31.7 mm to (145.4, 130.4), turned to 180 degrees
- moved R3 29.7 mm to (132.5, 108.0)
- moved R10 28.5 mm to (145.4, 128.4), turned to 180 degrees
- moved U2 27.8 mm to (134.0, 114.0), turned to 0 degrees
- moved R5 24.1 mm to (136.5, 108.0)
- moved C11 20.6 mm to (148.6, 127.2)
- moved C9 20.6 mm to (150.9, 124.9)
- moved IC1 20.6 mm to (148.6, 124.7)
- moved U3 20.6 mm to (139.7, 128.4), turned to 0 degrees
- moved J5 20.1 mm to (157.1, 90.3)
- moved J2 20.0 mm to (157.1, 98.8)
- moved R4 18.3 mm to (150.9, 85.7), turned to 180 degrees
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Connections:
- net /CAN/CAN2_H renamed /CAN1/CAN2_H
- net /CAN/CAN2_L renamed /CAN1/CAN2_L
- net /SCL renamed /SCL1
- net /SDA renamed /SDA1
- C1 pad 1: /power/+24V_aft_filt -> GND
- C1 pad 2: GND -> +3V3
- C3 pad 2: +5V -> +3V3
- C8 pad 2: /CAN/OSC2 -> +3V3
- D6 pad 1: Net-(D6-K) -> GND
- D6 pad 2: +5V -> Net-(D6-A)
- D7 pad 1: Net-(D7-K) -> GND
- D7 pad 2: +3V3 -> Net-(D7-A)
- FL1 pad 1: /power/+24V_preCMfilter -> GNDPWR
- FL1 pad 2: GNDPWR -> /power/+24V_preCMfilter
- FL1 pad 3: GND -> /power/+24V_proCMfilter
- FL1 pad 4: /power/+24V_proCMfilter -> GND
- J1 pad 11: /P17 -> /SPI1 CE1
- J1 pad 12: unconnected-(J1-GPIO18/PWM0-Pad12) -> /SPI1 CE0
- J1 pad 13: /P27 -> unconnected-(J1-GPIO27-Pad13)
- J1 pad 15: /P22 -> /D22
- J1 pad 16: /P23 -> /D23
- J1 pad 18: /P24 -> /D24
- J1 pad 19: /MOSI0 -> /SPI0 MOSI
- J1 pad 21: /MISO0 -> /SPI0 MISO
- J1 pad 22: /P25 -> /D25
- J1 pad 23: /SCLK0 -> /SPI0 SCLK
- J1 pad 24: unconnected-(J1-~{CE0}/GPIO8-Pad24) -> /SPI0 CE0
- J1 pad 26: unconnected-(J1-~{CE1}/GPIO7-Pad26) -> /SPI0 CE1
- J1 pad 27: unconnected-(J1-ID_SD/GPIO0-Pad27) -> /SDA0
- J1 pad 28: unconnected-(J1-ID_SC/GPIO1-Pad28) -> /SCL0
- J1 pad 32: /PWM0 -> unconnected-(J1-PWM0/GPIO12-Pad32)
- J1 pad 33: /PWM1 -> /D13
- J1 pad 35: /MISO1 -> /SPI1 MISO
- J1 pad 36: /P16 -> /SPI1 CE2
- J1 pad 37: /P26 -> unconnected-(J1-GPIO26-Pad37)
- J1 pad 38: /MOSI1 -> /SPI1 MOSI
- J1 pad 40: /SCLK1 -> /SPI1 SCLK
- R11 pad 1: Net-(U2-~{RESET}) -> Net-(U12-~{RESET})
- R11 pad 2: +5V -> +3V3
- R12 pad 1: Net-(IC3-EN) -> /SCLK
- R12 pad 2: +3V3 -> /SPI0 SCLK
- R13 pad 1: Net-(D6-K) -> +5V
- R13 pad 2: GND -> Net-(D6-A)
- R14 pad 1: Net-(D7-K) -> +3V3
- R14 pad 2: GND -> Net-(D7-A)
- R3 pad 1: /CAN/CANOPEN_RUN_LED -> /SPI1 CE2
- R3 pad 2: Net-(D2-K) -> /IMU/IMU_SPI_CS
- R5 pad 1: /CAN/CANOPEN_ERR_LED -> /SPI1 MISO
- R5 pad 2: Net-(D4-K) -> /IMU/IMU_SPI_MISO
- R6 pad 1: Net-(U5-SDO/SA0) -> /SPI1 SCLK
- R6 pad 2: +3V3 -> /IMU/IMU_SPI_SCK
- R8 pad 1: /P24 -> /SCLK
- R8 pad 2: Net-(IC3-A4) -> /SPI1 SCLK
- U2 pad 1: /CAN/CANTX -> /IMU/IMU_SPI_MISO
- U2 pad 10: /CAN/RX1BF -> unconnected-(U2-OCS_AUX-Pad10)
- U2 pad 11: /CAN/RX0BF -> unconnected-(U2-SDO_AUX-Pad11)
- U2 pad 12: /CAN/INT -> /IMU/IMU_SPI_CS
- U2 pad 13: /MCP2515_SCK -> /IMU/IMU_SPI_SCK
- U2 pad 14: /MCP2515_MOSI -> /IMU/IMU_SPI_MOSI
- U2 pad 2: /CAN/CANRX -> GND
- U2 pad 3: unconnected-(U2-CLKOUT/SOF-Pad3) -> GND
- U2 pad 4: /CAN/TX0RTS -> unconnected-(U2-INT1-Pad4)
- U2 pad 5: /CAN/TX1RTS -> +3V3
- U2 pad 6: /CAN/TX2RTS -> GND
- U2 pad 7: /CAN/OSC2 -> GND
- U2 pad 8: /CAN/OSC1 -> +3V3
- U2 pad 9: GND -> unconnected-(U2-INT2-Pad9)
- U4 pad 1: /CAN/CANTX -> /CAN1/CANTX
- U4 pad 4: /CAN/CANRX -> /CAN1/CANRX
- U5 pad 12: +3V3 -> Net-(U5-CS)
- U5 pad 4: /IMU/LSM6D_INT1 -> unconnected-(U5-INT1-Pad4)
- U5 pad 9: /IMU/LSM6D_INT2 -> unconnected-(U5-INT2-Pad9)
- Y2 pad 1: /CAN/OSC1 -> /CAN1/OSC1
- Y2 pad 2: /CAN/OSC2 -> GND
Routing:
- net +5V: track 82.8 -> 177.6 mm, vias 5 -> 0
- net /SPI1 SCLK: track 0.00 -> 45.1 mm, vias 0 -> 2
- net /SPI1 MOSI: track 0.00 -> 44.2 mm, vias 0 -> 2
- net /SPI1 CE2: track 0.00 -> 42.6 mm, vias 0 -> 2
- net /CAN0_INT: track 0.00 -> 41.1 mm
- net /CE0: track 0.00 -> 40.7 mm
- net /SPI1 MISO: track 0.00 -> 40.2 mm, vias 0 -> 3
- net /MISO: track 0.00 -> 39.4 mm
- net /MOSI: track 0.00 -> 38.7 mm
- net +3V3: track 143.2 -> 179.6 mm, vias 3 -> 9
- net /SCLK: track 0.00 -> 33.6 mm, vias 0 -> 2
- net /D13: track 0.00 -> 26.8 mm
- net /SDA1: track 59.8 -> 84.4 mm, vias 2 -> 5
- net /CE1: track 0.00 -> 22.9 mm, vias 0 -> 2
- net /CAN0/CAN2_L: track 0.00 -> 22.5 mm
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- added copper zone on In1.Cu, net GND
- added copper zone on In2.Cu, net GND
- removed copper zone on B.Cu, net GND
Other:
- copper layers 2 -> 4
- board text added: "- 24V +"
- board text added: "0 1"
- board text added: "1 0"
- board text added: "1.0 0.1"
- board text added: "1.1 0.0"
- board text added: "23 22"
- board text added: "24 25 13"
- board text added: "CAN0"
- board text added: "CAN1"
- board text added: "CE0"
- board text added: "CE1"
- board text added: "D36"
- board text added: "EP6 RPI_diyhat1 V1.2 25/08/14 Jack Kuo"
- board text added: "I2C1"
- board text added: "INT0"
- board text added: "INT1"
- board text added: "L H"
- board text added: "LSM303AGR"
- board text added: "MISO"
- board text added: "MOSI"
- board text added: "SCK"
- board text added: "SCLK"
- board text added: "SPI1"
- board text removed: "+ 24V -"
- board text removed: "EP6 RPI_diyhat1 V1.0 25/06/30 Jack Kuo"
- board text removed: "L CAN H"
- board text removed: "LSM303AGRTR"
