File: EP7/Electrical_Group/VCU_CM5/CAN.kicad_sch (KiCad schematic)
At the start: 9 parts, among them J25 CAN, U13 TCAN1042VDRQ1

Commit message: VCU_CM5 initial floorplan
Parts:
- J5: renamed from J25; footprint Connector_JST:JST_XH_B2B-XH-A_1x02_P2.50mm_Vertical -> Connector_JST:JST_PH_B2B-PH-K_1x02_P2.00mm_Vertical
- renumbered C123 to C22, C124 to C23, D38 to D4, R136 to R10, R137 to R11, R138 to R12, U13 to U3
Connections:
- net CAN-: now reaches FL2.3, J5.1 (Pin_1)
- net CAN-: now also D4.2 (K); no longer D4.1 (K)
- net CAN+: now reaches FL2.4, J5.2 (Pin_2)
- net CAN+: now also D4.1 (K); no longer D4.2 (K)
Other:
- moved on the sheet: J5
