File: EP7/Electrical_Group/VCU_CM5/stlink.kicad_sch (KiCad schematic)
At the start: 31 parts, among them J7 S_SWD, Q2 MMBT3904, U5 STM32F103CBT6, Y1 8MHz X50328MSB2GI

Commit message: VCU_CM5 initial floorplan
Parts:
- renumbered C37 to C35, C38 to C36, C39 to C37, C40 to C38, C41 to C39, C42 to C40, C43 to C41, C44 to C42, J7 to J6, R37 to R39, R38 to R40, R39 to R41, R40 to R42, R41 to R43, R42 to R44, R43 to R45, R44 to R46, R45 to R47, R46 to R48, R47 to R49, R48 to R50, R49 to R51, R50 to R52, R51 to R53, R52 to R54, R53 to R55
