File: EP7/Electrical_Group/VCU_CM5/vcu_mcu.kicad_sch (KiCad schematic)
At the start: 77 parts, among them J22 USART6, J23 MSD-4-A, Q3 2N7002, Q4 2N7002, Q5 AO3401A, SW2 RESET, SW3 BOOT0, U10 SN74LVC4245APWR, U11 STM32H743ZITx, Y3 8MHz X50328MSB2GI, Y4 32.768kHz Q13FC13500004

Commit message: VCU_CM5 initial floorplan
Parts:
- removed Q4: 2N7002, Package_TO_SOT_SMD:SOT-23, symbol Transistor_FET:2N7002
- removed Q5: AO3401A, Package_TO_SOT_SMD:SOT-23, symbol Transistor_FET:AO3401A
- removed R118, R120: 1k, Resistor_SMD:R_0603_1608Metric, symbol Device:R_Small
- removed R119: 10k, Resistor_SMD:R_0603_1608Metric, symbol Device:R_Small
- added J12: Conn_02x16_Odd_Even, Connector_PinSocket_2.00mm:PinSocket_2x16_P2.00mm_Vertical, symbol Connector_Generic:Conn_02x16_Odd_Even
- renumbered C102 to C100, C103 to C101, C104 to C102, C105 to C103, C106 to C104, C107 to C105, C108 to C106, C84 to C82, C85 to C83, C86 to C84, C87 to C85, C88 to C86, C89 to C87, C90 to C88, C91 to C89, C92 to C90, C93 to C91, C94 to C92, C95 to C93, C96 to C94, C97 to C95, C98 to C96, C99 to C97, C100 to C98, C101 to C99, J22 to J13, J23 to J14, R98 to R100, R99 to R101, R100 to R102, R101 to R103, R102 to R104, R103 to R105, R104 to R106, R105 to R107, R106 to R108, R107 to R109, R108 to R110, R110 to R111, R111 to R112, R112 to R113, R113 to R114, R114 to R115, R115 to R116, R116 to R117, R117 to R118, R121 to R119, R122 to R120, R123 to R121, R124 to R122, R125 to R123, R126 to R124, R127 to R125, R128 to R126, R129 to R127, R95 to R97, R96 to R98, R97 to R99
